File: hardware/KiCAD/ESP32_controler/ESP32_controler.kicad_pcb (KiCad board)
At the start: 2 copper layers, 20 parts, among them J1 Conn_01x15, J2 Conn_01x15, Q1 IRF540N, Q2 IRF540N, Q3 IRF540N

Commit message: edited Kicad schematics
Parts:
- +15V1, +48V1, Laser-A1, Laser-B1: footprint Connector_PinHeader_2.54mm:PinHeader_1x02_P2.54mm_Vertical -> TerminalBlock_Phoenix:TerminalBlock_Phoenix_MKDS-1,5-2-5.08_1x02_P5.08mm_Horizontal
- moved Laser-A1 13.3 mm to (72.5, 97.4), turned to -90 degrees
- moved +15V1 11.2 mm to (152.5, 65.0), turned to 180 degrees
- moved +48V1 10.3 mm to (97.5, 65.0), turned to 180 degrees
- moved Laser-B1 10.2 mm to (72.5, 110.0), turned to -90 degrees
- moved H2 2.50 mm to (162.5, 67.5)
Routing:
- net Net-(J1-Pin_2): track 94.5 -> 126.1 mm, vias 0 -> 4
- net Net-(+15V1-Pin_2): track 0.00 -> 26.5 mm
- net Net-(Laser-A1-Pin_1): track 10.5 -> 23.3 mm
- net Net-(Laser-B1-Pin_1): track 10.4 -> 21.3 mm
- net Net-(+48V1-Pin_2): track 16.6 -> 27.4 mm
- net Net-(+48V1-Pin_1): track 28.0 -> 19.9 mm
- net Net-(+15V1-Pin_1): track 56.7 -> 61.7 mm
- net Net-(J1-Pin_8): track 55.5 -> 56.3 mm
Other:
- board text added: "Laser-A2"
