File: hardware/KiCAD/ADC_controler/JTS - Controleur V4.kicad_pcb (KiCad board)
At the start: 2 copper layers, 119 x 114 mm, 22 parts, among them J4 Analog in, Q1 Q_NMOS_DGS, Q2 Q_NMOS_DGS, U1 AD797

Commit message: edited Kicad schematics
Parts:
- added J6: Analog GND, TerminalBlock_Phoenix:TerminalBlock_Phoenix_MKDS-1,5-2-5.08_1x02_P5.08mm_Horizontal, F.Cu at (177.5, 52.5)
- J1: renamed from Power In; value Conn_01x08_Pin -> Power in
- J5: renamed from Power Out; value Conn_01x08_Pin -> Power out
- Q1, Q2: footprint Package_TO_SOT_THT:TO-218-3_Vertical -> Package_TO_SOT_THT:TO-220-3_Vertical
- moved R7 40.3 mm to (147.5, 120.0), turned to 180 degrees
Connections:
- J1 pad 2: Earth -> Net-(J1-Pin_2)
- J5 pad 7: Earth -> Net-(J1-Pin_2)
- Q2 pad 1: Net-(J5-Pin_2) -> Net-(Q2-D)
- Q2 pad 3: Net-(Q2-S) -> Net-(J1-Pin_2)
- R2 pad 1: Earth -> Net-(J6-Pin_1)
- R7 pad 1: Earth -> Net-(J5-Pin_2)
- R7 pad 2: Net-(Q2-S) -> Net-(Q2-D)
Routing:
- net Net-(J1-Pin_2): track 0.00 -> 100.7 mm, vias 0 -> 2
- net Net-(J6-Pin_1): track 0.00 -> 58.6 mm, vias 0 -> 1
- net Net-(Q2-D): track 0.00 -> 27.7 mm, vias 0 -> 2
- net Net-(J5-Pin_2): track 71.7 -> 59.6 mm
- net Net-(Q2-S): track 11.4 -> 0.00 mm
- net Net-(Q1-S): track 69.0 -> 63.2 mm
- net Net-(Q2-G): track 18.1 -> 13.5 mm, vias 1 -> 0
- net Net-(Q1-G): track 64.6 -> 61.1 mm

Commit message: edited Kicad schematics
Parts:
- added Q3: Q_NMOS_DGS, Package_TO_SOT_THT:TO-220-3_Vertical, F.Cu at (160.0, 92.5)
- added R8: R, Resistor_THT:R_Axial_DIN0309_L9.0mm_D3.2mm_P15.24mm_Horizontal, F.Cu at (172.6, 77.5)
- added SAturating: Saturating Pulse, TerminalBlock_Phoenix:TerminalBlock_Phoenix_MKDS-1,5-2-5.08_1x02_P5.08mm_Horizontal, F.Cu at (150.0, 52.5)
- Analog GND: renamed from J6
- Analog In: renamed from J4
Routing:
- net Net-(J7-Pin_1): track 0.00 -> 51.0 mm, vias 0 -> 2
- net Net-(J6-Pin_1): track 58.6 -> 89.6 mm, vias 1 -> 2
- net Net-(Q3-S): track 0.00 -> 22.6 mm, vias 0 -> 1
- net Net-(Q1-S): track 63.2 -> 78.5 mm
